Commit message: Fixed urdf

File: urdf/example.urdf (robot description, URDF)
Before this commit: robot myfirst, 3 links, 2 joints
Links:
- removed link Left_wheel
- removed link Right_wheel
- added link left_wheel; visual cylinder length=0.02 radius=0.05
- added link right_wheel; visual cylinder length=0.02 radius=0.05
- link base_link: geometry visual cylinder length=0.1 radius=0.1
Joints:
- removed joint Left
- removed joint Right
- added joint left_joint: type continuous, parent base_link, child left_wheel, origin xyz=0 0.1 0.05 rpy=1.57075 0.0 0.0, axis 0 0 -1, limit effort=2 velocity=10
- added joint right_joint: type continuous, parent base_link, child right_wheel, origin xyz=0 -0.1 0.05 rpy=1.57075 0.0 0.0, axis 0 0 1, limit effort=2 velocity=10

Commit message: Setup urdf and other files

File: urdf/example.urdf (robot description, URDF)
Before this commit: robot example, 3 links, 2 joints
Links:
- link left_wheel: geometry collision cylinder length=0.02 radius=0.05; visual cylinder length=0.02 radius=0.05
- link right_wheel: geometry collision cylinder length=0.02 radius=0.05; visual cylinder length=0.02 radius=0.05
Joints:
- joint right_joint: axis 0 0 1 -> 0 0 -1
